Commit message: - Feature  : Files added

File: ur_robot/urdf/small_bin/bin.urdf (robot description, URDF)
Before this commit: robot bin, 6 links, 5 joints
Links:
- link back: geometry collision box size=0.4 0.02 0.1; visual box size=0.4 0.02 0.1
- link front: geometry collision box size=0.4 0.02 0.1; visual box size=0.4 0.02 0.1
- link left: geometry collision box size=0.02 0.4 0.1; visual box size=0.02 0.4 0.1
- link right: geometry collision box size=0.02 0.4 0.1; visual box size=0.02 0.4 0.1
